Commit message: reset wrist angle

File: wam_description/urdf/wam_finger.urdf (robot description, URDF)
Before this commit: robot wam, 20 links, 19 joints
Joints:
- joint wam_joint_7: limit lower=-1.5 upper=1.5 effort=30 velocity=2.0 -> lower=-3.0 upper=3.0 effort=30 velocity=2.0

Commit message: add comment for fixing bhand spread & adjust wrist angle

File: wam_description/urdf/wam_finger.urdf (robot description, URDF)
Before this commit: robot wam, 20 links, 19 joints
Joints:
- joint wam_joint_7: limit lower=-3.0 upper=3.0 effort=30 velocity=2.0 -> lower=-1.5 upper=1.5 effort=30 velocity=2.0

Commit message: Reworked corner reward calculations to be much more accurate Removed height penalty since it has been restricted

File: wam_description/urdf/wam_finger.urdf (robot description, URDF)
Before this commit: robot wam, 20 links, 19 joints
Links:
- link bhand_finger1_link_3: geometry collision box size=0.066 0.019 0.023; visual box size=0.1 0.02 0.02
- link bhand_finger2_link_3: geometry collision box size=0.066 0.019 0.023; visual box size=0.1 0.02 0.02
- link bhand_finger3_link_3: geometry collision box size=0.066 0.019 0.023; visual box size=0.1 0.02 0.02
